File: hardware/kicad/JECCbotECU.kicad_pcb (KiCad board)
At the start: 2 copper layers, 59 parts, among them CN1 ADAFRUIT_FEATHER, CN2 691382010004, CN3 691382010005, CN4 691382010004, P1 USB_B, P2 CONN_02X05, P3 CONN_02X03, U1 STM32F103C8Tx, U2 BSS138, U3 BSS138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

Commit message: started pcb
Parts:
- added MH1: MH_210_400_NP, MECH_mounting_holes:MH_210_400_NP, F.Cu at (93.0, 43.0)
- added MH2: MH_210_400_NP, MECH_mounting_holes:MH_210_400_NP, F.Cu at (187.0, 43.0)
- added MH3: MH_210_400_NP, MECH_mounting_holes:MH_210_400_NP, F.Cu at (93.0, 97.0)
- added MH4: MH_210_400_NP, MECH_mounting_holes:MH_210_400_NP, F.Cu at (187.0, 97.0)
- added P4: CONN_02X05, pin_headers:Pin_Header_Angled_2x05, F.Cu at (175.3, 67.3)
- moved P3 126.2 mm to (175.3, 85.1)
- moved P1 125.3 mm to (158.8, 83.8), turned to 270 degrees
- moved C19 122.6 mm to (37.4, 123.1), turned to 180 degrees
- moved C11 118.5 mm to (35.0, 117.0), turned to 180 degrees
- moved R16 118.4 mm to (31.2, 114.4), turned to 180 degrees
- moved P2 117.9 mm to (175.3, 49.5)
- moved C22 110.5 mm to (39.8, 116.6), turned to 180 degrees
- moved U5 110.3 mm to (44.5, 121.5), turned to 180 degrees
- moved R6 109.4 mm to (155.6, 120.9)
- moved U2 107.6 mm to (147.9, 118.0)
- moved R5 106.3 mm to (162.9, 118.2)
- moved R18 106.2 mm to (38.2, 110.9), turned to 180 degrees
- moved R14 106.1 mm to (40.1, 113.6), turned to 180 degrees
- moved R3 100.2 mm to (159.2, 118.2)
- moved R8 98.9 mm to (151.9, 119.8)
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Connections:
- U1 pad 10: Net-(U1-Pad10) -> GPIO
- U1 pad 39: Net-(U1-Pad39) -> SPI_SCK
- U1 pad 40: Net-(U1-Pad40) -> SPI_MISO
- U1 pad 41: Net-(U1-Pad41) -> SPI_MOSI
Other:
- board outline added: 100 x 60 mm

Commit message: component placement almost done
Parts:
- removed X1: 8MHz, crystals:Crystal_HC49-U_Vertical
- added Y1: Crystal_Small, crystals:Crystal_HC49-U_Vertical, F.Cu at (157.5, 55.9)
- moved C5 135.6 mm to (160.0, 50.8), turned to 270 degrees
- moved C11 132.3 mm to (149.5, 50.8), turned to 0 degrees
- moved R1 131.8 mm to (157.5, 59.7)
- moved C6 130.4 mm to (154.9, 50.8), turned to 90 degrees
- moved C2 128.8 mm to (166.4, 67.3)
- moved R14 127.2 mm to (149.3, 48.3), turned to 0 degrees
- moved U1 125.0 mm to (157.5, 69.8), turned to 270 degrees
- moved U5 121.6 mm to (143.5, 50.8), turned to 0 degrees
- moved R18 121.1 mm to (146.1, 55.9), turned to 90 degrees
- moved C23 120.5 mm to (145.8, 45.7), turned to 0 degrees
- moved R15 119.6 mm to (149.3, 55.9)
- moved C1 117.1 mm to (151.9, 62.2), turned to 180 degrees
- moved R19 116.7 mm to (143.5, 55.9), turned to 270 degrees
- moved C21 112.7 mm to (145.8, 43.2), turned to 0 degrees
- moved C4 112.3 mm to (160.0, 78.7), turned to 270 degrees
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Connections:
- U1 pad 3: OSC_IN -> Net-(U1-Pad3)
- U1 pad 4: OSC_OUT -> Net-(U1-Pad4)
- U1 pad 5: Net-(U1-Pad5) -> OSC_IN
- U1 pad 6: Net-(U1-Pad6) -> OSC_OUT

Commit message: pcb placement
Parts:
- moved C9 95.4 mm to (97.7, 68.2)
- moved R12 95.4 mm to (98.7, 73.4)
- moved C7 95.4 mm to (93.5, 72.4)
- moved R13 95.4 mm to (101.5, 68.3)
- moved C8 76.6 mm to (104.1, 74.9)
- moved C10 67.5 mm to (105.4, 72.4)
- moved R5 66.5 mm to (170.2, 52.1)
- moved R6 64.1 mm to (170.2, 58.4)
- moved R2 39.9 mm to (149.9, 78.7), turned to 270 degrees
- moved R3 39.9 mm to (153.7, 78.7), turned to 90 degrees
- moved R4 23.8 mm to (157.5, 78.7), turned to 90 degrees
Changed lines of the file:
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@@
   )
   (module resistors:R_0603 (layer F.Cu)
-    (at 58.33 153.39)
+    (at 101.51 68.3)
     (descr "Resistor SMD 0603, reflow soldering, Vishay (see dcrcw.pdf)")
     (tags "resistor 0603")
@@
   )
   (module resistors:R_0603 (layer F.Cu)
-    (at 55.48 158.49)
+    (at 98.66 73.4)
     (descr "Resistor SMD 0603, reflow soldering, Vishay (see dcrcw.pdf)")
     (tags "resistor 0603")
@@
   )
   (module resistors:R_0603 (layer F.Cu)
-    (at 155.58 120.86)
+    (at 170.18 58.42)
     (descr "Resistor SMD 0603, reflow soldering, Vishay (see dcrcw.pdf)")
     (tags "resistor 0603")
@@
   )
   (module resistors:R_0603 (layer F.Cu)
-    (at 162.88 118.21)
+    (at 170.18 52.07)
     (descr "Resistor SMD 0603, reflow soldering, Vishay (see dcrcw.pdf)")
     (tags "resistor 0603")
@@
   )
   (module resistors:R_0603 (layer F.Cu)
-    (at 145.1 99.05)
+    (at 157.48 78.74 90)
     (descr "Resistor SMD 0603, reflow soldering, Vishay (see dcrcw.pdf)")
     (tags "resistor 0603")
     (attr smd)
-    (fp_text reference R4 (at 0 -1.9) (layer F.SilkS)
-      (effects (font (size 1 1) (thickness 0.15)))
-    )
-    (fp_text value 4.7k (at 0 1.9) (layer F.Fab)
+    (fp_text reference R4 (at 0 -1.27 90) (layer F.SilkS)
+      (effects (font (size 1 1) (thickness 0.15)))
+    )
+    (fp_text value 4.7k (at 0 1.9 90) (layer F.Fab)
       (effects (font (size 1 1) (thickness 0.15)))
     )
@@
     (fp_line (start -1.3 0.8) (end 1.3 0.8) (layer F.CrtYd) (width 0.05))
     (fp_line (start -1.3 -0.8) (end 1.3 -0.8) (layer F.CrtYd) (width 0.05))
-    (pad 2 smd rect (at 0.75 0) (size 0.5 0.9) (layers F.Cu F.Paste F.Mask)
+    (pad 2 smd rect (at 0.75 0 90) (size 0.5 0.9) (layers F.Cu F.Paste F.Mask)
       (net 13 +5V))
-    (pad 1 smd rect (at -0.75 0) (size 0.5 0.9) (layers F.Cu F.Paste F.Mask)
+    (pad 1 smd rect (at -0.75 0 90) (size 0.5 0.9) (layers F.Cu F.Paste F.Mask)
       (net 64 USB+))
     (model resistors.3dshapes/R_0603.wrl
@@
   )
   (module resistors:R_0603 (layer F.Cu)
-    (at 159.23 118.21)
+    (at 153.67 78.74 90)
     (descr "Resistor SMD 0603, reflow soldering, Vishay (see dcrcw.pdf)")
     (tags "resistor 0603")
     (attr smd)
-    (fp_text reference R3 (at 0 -1.9) (layer F.SilkS)
-      (effects (font (size 1 1) (thickness 0.15)))
-    )
-    (fp_text value 20 (at 0 1.9) (layer F.Fab)
+    (fp_text reference R3 (at 0 -1.27 90) (layer F.SilkS)
+      (effects (font (size 1 1) (thickness 0.15)))
+    )
+    (fp_text value 20 (at 0 1.9 90) (layer F.Fab)
       (effects (font (size 1 1) (thickness 0.15)))
     )
@@
     (fp_line (start -1.3 0.8) (end 1.3 0.8) (layer F.CrtYd) (width 0.05))
     (fp_line (start -1.3 -0.8) (end 1.3 -0.8) (layer F.CrtYd) (width 0.05))
-    (pad 2 smd rect (at 0.75 0) (size 0.5 0.9) (layers F.Cu F.Paste F.Mask)
+    (pad 2 smd rect (at 0.75 0 90) (size 0.5 0.9) (layers F.Cu F.Paste F.Mask)
       (net 64 USB+))
-    (pad 1 smd rect (at -0.75 0) (size 0.5 0.9) (layers F.Cu F.Paste F.Mask)
+    (pad 1 smd rect (at -0.75 0 90) (size 0.5 0.9) (layers F.Cu F.Paste F.Mask)
       (net 47 "Net-(P1-Pad3)"))
     (model resistors.3dshapes/R_0603.wrl
@@
   )
   (module resistors:R_0603 (layer F.Cu)
-    (at 155.58 118.21)
+    (at 149.86 78.74 270)
     (descr "Resistor SMD 0603, reflow soldering, Vishay (see dcrcw.pdf)")
     (tags "resistor 0603")
     (attr smd)
-    (fp_text reference R2 (at 0 -1.9) (layer F.SilkS)
-      (effects (font (size 1 1) (thickness 0.15)))
-    )
-    (fp_text value 20 (at 0 1.9) (layer F.Fab)
+    (fp_text reference R2 (at 0 1.27 90) (layer F.SilkS)
+      (effects (font (size 1 1) (thickness 0.15)))
+    )
+    (fp_text value 20 (at 0 1.9 90) (layer F.Fab)
       (effects (font (size 1 1) (thickness 0.15)))
     )
@@
     (fp_line (start -1.3 0.8) (end 1.3 0.8) (layer F.CrtYd) (width 0.05))
     (fp_line (start -1.3 -0.8) (end 1.3 -0.8) (layer F.CrtYd) (width 0.05))
-    (pad 2 smd rect (at 0.75 0) (size 0.5 0.9) (layers F.Cu F.Paste F.Mask)
+    (pad 2 smd rect (at 0.75 0 270) (size 0.5 0.9) (layers F.Cu F.Paste F.Mask)
       (net 48 "Net-(P1-Pad2)"))
-    (pad 1 smd rect (at -0.75 0) (size 0.5 0.9) (layers F.Cu F.Paste F.Mask)
+    (pad 1 smd rect (at -0.75 0 270) (size 0.5 0.9) (layers F.Cu F.Paste F.Mask)
       (net 63 USB-))
     (model resistors.3dshapes/R_0603.wrl
@@
   )
   (module capacitors:C_0603 (layer F.Cu)
-    (at 100.33 139.7)
+    (at 105.41 72.39)
     (descr "Capacitor SMD 0603, reflow soldering, AVX (see smccp.pdf)")
     (tags "capacitor 0603")
@@
   )
   (module capacitors:C_0603 (layer F.Cu)
-    (at 54.53 153.34)
+    (at 97.71 68.25)
     (descr "Capacitor SMD 0603, reflow soldering, AVX (see smccp.pdf)")
     (tags "capacitor 0603")
@@
   )
   (module capacitors:C_0603 (layer F.Cu)
-    (at 96.13 151.12)
+    (at 104.14 74.93)
     (descr "Capacitor SMD 0603, reflow soldering, AVX (see smccp.pdf)")
     (tags "capacitor 0603")
@@
   )
   (module capacitors:C_0603 (layer F.Cu)
-    (at 50.28 157.48)
+    (at 93.46 72.39)
     (descr "Capacitor SMD 0603, reflow soldering, AVX (see smccp.pdf)")
     (tags "capacitor 0603")
@@
     (tags "capacitor 0603")
     (attr smd)
-    (fp_text reference C4 (at 0 -1.9 90) (layer F.SilkS)
-      (effects (font (size 1 1) (thickness 0.15)))
-    )
+    (fp_text reference C4 (at 0 -1.27 90) (layer F.SilkS)
+      (effects (font (size 1 1) (thickness 0.15)))
+    )

Commit message: finished component placement
Parts:
- moved C7 25.9 mm to (119.4, 72.4), turned to 270 degrees
- moved R12 23.3 mm to (121.9, 72.4), turned to 90 degrees
- moved C9 17.4 mm to (114.3, 73.7)
- moved C3 16.3 mm to (149.3, 69.8), turned to 180 degrees
- moved C8 13.5 mm to (114.3, 66.0)
- moved R13 13.2 mm to (114.5, 71.1)
- moved C10 9.67 mm to (114.3, 68.6)
- moved U4 6.48 mm to (120.7, 67.3)
- moved R1 3.59 mm to (160.0, 57.1)
- moved Y1 3.59 mm to (160.0, 53.3)
- moved U1 3.59 mm to (160.0, 67.3)
- moved C2 3.59 mm to (168.9, 64.8)
- moved C1 3.59 mm to (154.4, 59.7)
- moved C5 3.59 mm to (162.6, 48.3)
- moved C6 3.59 mm to (157.5, 48.3)
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
Commit message: finished layout
Parts:
- removed C18: DNI, capacitors:C_1210
- added C24: 10uF, capacitors:C_0603, F.Cu at (167.6, 43.2)
- added C25: 22uF, capacitors:C_0603, F.Cu at (167.6, 48.3)
- added P5: WR-TBL_691313710002, mechanical-connectors:WR-TBL_691313710002, F.Cu at (99.1, 69.8)
- added R20: 10k, resistors:R_0603, F.Cu at (108.2, 75.2)
- added R21: 10k, resistors:R_0603, F.Cu at (108.2, 71.4)
- added U7: LT1117, SOT_TO:SOT-223, F.Cu at (157.5, 45.7)
- moved C8 11.3 mm to (120.9, 75.2), turned to 180 degrees
- moved R12 9.34 mm to (113.3, 68.8), turned to 270 degrees
- moved C9 8.99 mm to (120.9, 67.6), turned to 180 degrees
- moved U4 8.99 mm to (114.6, 73.9), turned to 180 degrees
- moved C10 8.98 mm to (122.4, 72.5)
- moved R13 6.39 mm to (120.8, 70.1), turned to 180 degrees
- moved C7 5.03 mm to (115.8, 68.8), turned to 90 degrees
- moved C5 4.02 mm to (163.8, 52.1)
- moved C6 4.02 mm to (158.8, 52.1), turned to 270 degrees
- moved R1 4.02 mm to (161.3, 61.0)
- moved Y1 4.02 mm to (161.3, 57.1)
- moved R6 3.97 mm to (173.2, 55.8)
- moved C1 3.31 mm to (157.5, 61.0)
- moved C3 3.19 mm to (150.9, 72.6)
- moved R2 3.05 mm to (152.9, 78.7)
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Connections:
- C12 pad 1: +12V -> VBAT
- C14 pad 1: +12V -> VBAT
- C15 pad 2: Net-(C15-Pad2) -> GND
- C16 pad 2: Net-(C15-Pad2) -> GND
- CN1 pad 11: Net-(CN1-Pad11) -> SPI_SCK
- CN1 pad 12: Net-(CN1-Pad12) -> SPI_MOSI
- CN1 pad 13: Net-(CN1-Pad13) -> SPI_MISO
- R17 pad 2: Net-(C15-Pad2) -> GND
- U5 pad 2: +12V -> VBAT
- U6 pad 1: Net-(C15-Pad2) -> GND
Routing:
- net +3V3: track 0.00 -> 328.4 mm, vias 0 -> 6
- net +5V: track 0.00 -> 256.5 mm, vias 0 -> 2
- net +12V: track 0.00 -> 170.5 mm, vias 0 -> 1
- net I2C_SDA: track 0.00 -> 115.9 mm, vias 0 -> 1
- net I2C_SCL: track 0.00 -> 107.0 mm, vias 0 -> 1
- net LIDAR_PWM: track 0.00 -> 81.1 mm, vias 0 -> 1
- net SPI_SCK: track 0.00 -> 80.2 mm, vias 0 -> 2
- net SPI_MISO: track 0.00 -> 74.1 mm, vias 0 -> 1
- net RESET: track 0.00 -> 73.9 mm, vias 0 -> 2
- net VBAT: track 0.00 -> 73.3 mm, vias 0 -> 1
- net SPI_MOSI: track 0.00 -> 69.4 mm, vias 0 -> 1
- net KVH_TX: track 0.00 -> 67.8 mm, vias 0 -> 2
- net LIDAR_RX: track 0.00 -> 67.8 mm, vias 0 -> 2
- net LIDAR_TX: track 0.00 -> 64.5 mm, vias 0 -> 2
- net KVH_RX: track 0.00 -> 63.8 mm, vias 0 -> 2
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- added copper zone on B.Cu, net GND
- added copper zone on F.Cu, net GND
Other:
- rule via_min_size: 0.4 -> 0.8
