File: hardware/kicad/JECCbotECU.sch (KiCad schematic (older format))
At the start: 9 parts, among them U1 STM32F103C8Tx, X1 8MHz

Commit message: bugfix
Connections:
- net GND: now also C5.1, C6.1
Other:
- moved on the sheet: C5, C6, R1, X1
Changed lines of the file:
@@
 INH34
 Text Label 1550 1900 0    60   ~ 0
-RESET
+NRST
 Wire Wire Line
 	1250 2800 2000 2800
@@
 L devices:QUARTZCMS4 X1
 U 1 1 5E89B855
-P 10300 2900
-F 0 "X1" H 10300 3255 50  0000 C CNN
-F 1 "8MHz" H 10300 3164 50  0000 C CNN
-F 2 "crystals:Crystal_HC49-U_Vertical" H 10300 3073 50  0000 C CNN
-F 3 "" H 10300 2900 50  0000 C CNN
-	1    10300 2900
-	1    0    0    -1
+P 10100 4000
+F 0 "X1" H 10100 4355 50  0000 C CNN
+F 1 "8MHz" H 10100 4264 50  0000 C CNN
+F 2 "crystals:Crystal_HC49-U_Vertical" H 10100 4173 50  0000 C CNN
+F 3 "" H 10100 4000 50  0000 C CNN
+	1    10100 4000
+	1    0    0    1
 $EndComp
 $Comp
 L devices:R_0603 R1
 U 1 1 5E89DE18
-P 10300 3350
-F 0 "R1" V 10104 3350 50  0000 C CNN
-F 1 "1M" V 10195 3350 50  0000 C CNN
-F 2 "resistors:R_0603" H 10300 3200 50  0001 C CNN
-F 3 "" H 10300 3350 50  0000 C CNN
-	1    10300 3350
-	0    1    1    0
+P 10100 3550
+F 0 "R1" V 9904 3550 50  0000 C CNN
+F 1 "1M" V 9995 3550 50  0000 C CNN
+F 2 "resistors:R_0603" H 10100 3400 50  0001 C CNN
+F 3 "" H 10100 3550 50  0000 C CNN
+	1    10100 3550
+	0    1    -1   0
 $EndComp
 $Comp
 L devices:C_0603 C5
 U 1 1 5E89FD98
-P 10000 2350
-F 0 "C5" H 10092 2396 50  0000 L CNN
-F 1 "20pF" H 10092 2305 50  0000 L CNN
-F 2 "capacitors:C_0603" H 10000 2200 50  0001 C CNN
-F 3 "" H 10000 2350 50  0000 C CNN
-	1    10000 2350
-	1    0    0    -1
+P 9800 4550
+F 0 "C5" H 9892 4596 50  0000 L CNN
+F 1 "20pF" H 9892 4505 50  0000 L CNN
+F 2 "capacitors:C_0603" H 9800 4400 50  0001 C CNN
+F 3 "" H 9800 4550 50  0000 C CNN
+	1    9800 4550
+	1    0    0    1
 $EndComp
 $Comp
 L devices:C_0603 C6
 U 1 1 5E8A00F6
-P 10600 2350
-F 0 "C6" H 10692 2396 50  0000 L CNN
-F 1 "20pF" H 10692 2305 50  0000 L CNN
-F 2 "capacitors:C_0603" H 10600 2200 50  0001 C CNN
-F 3 "" H 10600 2350 50  0000 C CNN
-	1    10600 2350
-	1    0    0    -1
-$EndComp
-Wire Wire Line
-	10000 2250 10000 2150
-Wire Wire Line
-	10000 2150 10600 2150
-Wire Wire Line
-	10600 2150 10600 2250
-Wire Wire Line
-	10600 2450 10600 2900
-Wire Wire Line
-	10000 2900 10000 2450
-Wire Wire Line
-	10000 2900 10000 3350
-Wire Wire Line
-	10000 3350 10200 3350
-Connection ~ 10000 2900
-Wire Wire Line
-	10400 3350 10600 3350
-Wire Wire Line
-	10600 3350 10600 2900
-Connection ~ 10600 2900
-Wire Wire Line
-	10600 3550 10600 3350
-Connection ~ 10600 3350
-Wire Wire Line
-	10000 3550 10000 3350
-Connection ~ 10000 3350
+P 10400 4550
+F 0 "C6" H 10492 4596 50  0000 L CNN
+F 1 "20pF" H 10492 4505 50  0000 L CNN
+F 2 "capacitors:C_0603" H 10400 4400 50  0001 C CNN
+F 3 "" H 10400 4550 50  0000 C CNN
+	1    10400 4550
+	1    0    0    1
+$EndComp
+Wire Wire Line
+	9800 4650 9800 4750
+Wire Wire Line
+	9800 4750 10100 4750
+Wire Wire Line
+	10400 4750 10400 4650
+Wire Wire Line
+	10400 4450 10400 4000
+Wire Wire Line
+	9800 4000 9800 4450
+Wire Wire Line
+	9800 4000 9800 3550
+Wire Wire Line
+	9800 3550 10000 3550
+Connection ~ 9800 4000
+Wire Wire Line
+	10200 3550 10400 3550
+Wire Wire Line
+	10400 3550 10400 4000
+Connection ~ 10400 4000
+Wire Wire Line
+	10400 3350 10400 3550
+Connection ~ 10400 3550
+Wire Wire Line
+	9800 3350 9800 3550
+Connection ~ 9800 3550
 Text GLabel 1500 3000 0    60   Output ~ 0
 OSC_OUT
-Text GLabel 10000 3550 3    50   Output ~ 0
+Text GLabel 9800 3350 1    50   Output ~ 0
 OSC_IN
-Text GLabel 10600 3550 3    50   Input ~ 0
+Text GLabel 10400 3350 1    50   Input ~ 0
 OSC_OUT
 $Sheet
@@
 NoConn ~ 2000 4600
 NoConn ~ 2000 4700
+$Comp
+L power-supply:GND #PWR?
+U 1 1 5E887774
+P 10100 4850
+F 0 "#PWR?" H 10100 4600 50  0001 C CNN
+F 1 "GND" H 10105 4677 50  0000 C CNN
+F 2 "" H 10100 4850 50  0000 C CNN
+F 3 "" H 10100 4850 50  0000 C CNN
+	1    10100 4850
+	-1   0    0    -1
+$EndComp
+Wire Wire Line
+	10100 4850 10100 4750
+Connection ~ 10100 4750
+Wire Wire Line
+	10100 4750 10400 4750
 $EndSCHEMATC

Commit message: finished schematics
Connections:
- net GPIO: now reaches U1.10 (ADC1_IN0/ADC2_IN0/SYS_WKUP/TIM2_CH1/TIM2_ETR/USART2_CTS/PA0)
- net SPI_SCK: now reaches U1.39 (PB3/SPI1_SCK/SYS_JTDO-TRACESWO/TIM2_CH2)
- net SPI_MISO: now reaches U1.40 (PB4/SPI1_MISO/SYS_NJTRST/TIM3_CH1)
- net SPI_MOSI: now reaches U1.41 (PB5/I2C1_SMBA/SPI1_MOSI/TIM3_CH2)
- no-connect marks 14 -> 10
Changed lines of the file:
@@
 Text Label 7900 3600 0    60   ~ 0
 INH34
-Wire Wire Line
-	8450 3600 7800 3600
-Wire Wire Line
-	8450 3700 7800 3700
-Wire Wire Line
-	1350 3300 2000 3300
-Wire Wire Line
-	1350 3200 2000 3200
-Wire Wire Line
-	8450 3900 7800 3900
-Wire Wire Line
-	8450 3800 7800 3800
 Text Label 7900 3900 0    60   ~ 0
 PWM3
@@
 Text Label 1900 3300 2    60   ~ 0
 PWM1
-Wire Wire Line
-	1350 3800 2000 3800
-Wire Wire Line
-	1350 3900 2000 3900
 Text Label 1900 3800 2    60   ~ 0
 I2C_SCL
@@
 Text GLabel 8450 3600 2    60   Output ~ 0
 INH34
-Text Label 1550 1900 0    60   ~ 0
-NRST
-Wire Wire Line
-	1250 2800 2000 2800
 Text GLabel 1250 2800 0    60   Input ~ 0
 EM_STOP_D
 Text Label 1300 2800 0    60   ~ 0
 EM_STOP_D
-Wire Wire Line
-	8550 3300 7800 3300
-Wire Wire Line
-	1500 1900 2000 1900
 Text Label 8500 3300 2    60   ~ 0
 VIN_MEAS
@@
 	4800 5250 4800 5100
 Wire Wire Line
-	5000 5100 5000 5250
-Wire Wire Line
 	5000 5250 4900 5250
 Connection ~ 4800 5250
-Wire Wire Line
-	4900 5100 4900 5250
 Connection ~ 4900 5250
 Wire Wire Line
@@
 Text GLabel 1350 4300 0    60   Input ~ 0
 GPS_RX
-Wire Wire Line
-	2000 2100 1500 2100
-Wire Wire Line
-	2000 4000 1350 4000
-Wire Wire Line
-	2000 4200 1350 4200
-Wire Wire Line
-	1350 4300 2000 4300
-Wire Wire Line
-	8450 4100 7800 4100
-Wire Wire Line
-	7800 4200 8450 4200
-Wire Wire Line
-	8450 4300 7800 4300
-Wire Wire Line
-	7800 4400 8450 4400
-Wire Wire Line
-	8450 3400 7800 3400
-Wire Wire Line
-	7800 3500 8450 3500
 Text GLabel 8450 4500 2    60   BiDi ~ 0
 SWDIO
@@
 Text GLabel 1500 2900 0    60   Input ~ 0
 OSC_IN
-Wire Wire Line
-	1350 3400 2000 3400
-Wire Wire Line
-	7800 4500 8450 4500
-Wire Wire Line
-	8450 4600 7800 4600
-Wire Wire Line
-	2000 2900 1500 2900
-Wire Wire Line
-	1500 3000 2000 3000
 $Sheet
 S 750  7050 1000 450
@@
 NoConn ~ 2000 2300
 $Sheet
-S 3050 7050 950  450
+S 4100 7050 950  450
 U 5E9A2887
 F0 "power" 50
@@
 $EndSheet
 $Sheet
-S 4150 7050 900  450
+S 3050 7050 900  450
 U 5E9DEA3D
 F0 "bno055" 50
 F1 "bno055.sch" 50
 $EndSheet
-NoConn ~ 7800 3200
 NoConn ~ 7800 4000
 NoConn ~ 7800 4700
 NoConn ~ 2000 2500
 NoConn ~ 2000 2600
-NoConn ~ 2000 3500
-NoConn ~ 2000 3600
-NoConn ~ 2000 3700
 NoConn ~ 2000 4100
 NoConn ~ 2000 4400
@@
 NoConn ~ 2000 4700
 $Comp
-L power-supply:GND #PWR?
+L power-supply:GND #PWR0116
 U 1 1 5E887774
 P 10100 4850
-F 0 "#PWR?" H 10100 4600 50  0001 C CNN
+F 0 "#PWR0116" H 10100 4600 50  0001 C CNN
 F 1 "GND" H 10105 4677 50  0000 C CNN
 F 2 "" H 10100 4850 50  0000 C CNN
@@
 Wire Wire Line
 	10100 4750 10400 4750
+Text GLabel 1350 3500 0    50   Output ~ 0
+SPI_SCK
+Wire Wire Line
+	7800 3600 8450 3600
+Wire Wire Line
+	7800 3700 8450 3700
+Wire Wire Line
+	7800 3900 8450 3900
+Wire Wire Line
+	7800 3800 8450 3800
+Wire Wire Line
+	7800 3300 8550 3300
+Wire Wire Line
+	7800 4100 8450 4100
+Wire Wire Line
+	7800 4200 8450 4200
+Wire Wire Line
+	7800 4300 8450 4300
+Wire Wire Line
+	7800 4400 8450 4400
+Wire Wire Line
+	7800 3400 8450 3400
+Wire Wire Line
+	7800 3500 8450 3500
+Wire Wire Line
+	7800 4500 8450 4500
+Wire Wire Line
+	7800 4600 8450 4600
+Wire Wire Line
+	5000 5100 5000 5250
+Wire Wire Line
+	4900 5100 4900 5250
+Text GLabel 1350 3600 0    50   Input ~ 0
+SPI_MISO
+Text GLabel 1350 3700 0    50   Output ~ 0
+SPI_MOSI
+Wire Wire Line
+	1350 3300 2000 3300
+Wire Wire Line
+	1350 3200 2000 3200
+Wire Wire Line
+	1350 3800 2000 3800
+Wire Wire Line
+	1350 3900 2000 3900
+Wire Wire Line
+	1250 2800 2000 2800
+Wire Wire Line
+	1500 1900 2000 1900
+Wire Wire Line
+	1500 2100 2000 2100
+Wire Wire Line
+	1350 4000 2000 4000
+Wire Wire Line
+	1350 4200 2000 4200
+Wire Wire Line
+	1350 4300 2000 4300
+Wire Wire Line
+	1350 3400 2000 3400
+Wire Wire Line
+	1500 2900 2000 2900
+Wire Wire Line
+	1500 3000 2000 3000
+Wire Wire Line
+	1350 3500 2000 3500
+Wire Wire Line
+	1350 3600 2000 3600
+Wire Wire Line
+	1350 3700 2000 3700
+Text GLabel 8450 3200 2    50   BiDi ~ 0
+GPIO
+Wire Wire Line
+	8450 3200 7800 3200
 $EndSCHEMATC

Commit message: started pcb
Other:
- note added: "JECCbot ECU"
- note removed: "Copyright generationmake 2019\nsee full project documentation at https://github.com/generationmake/HighPowerMotorFeatherWing"
- note removed: "You may redistribute and modify this documentation under the terms of the CERN OHL v.1.2. (http://ohwr.org/cernohl). \nThis documentation is distributed WITHOUT ANY EXPRESS OR IMPLIED WARRANTY, INCLUDING OF MERCHANTABILITY, SATISFACTORY \nQUALITY AND FITNESS FOR A PARTICULAR PURPOSE. Please see the CERN OHL v.1.2 for applicable conditions"
Changed lines of the file:
@@
 $EndDescr
 Text Notes 500  650  0    47   ~ 0
-Copyright generationmake 2019\nsee full project documentation at https://github.com/generationmake/HighPowerMotorFeatherWing
-Text Notes 7000 6900 0    43   ~ 0
-You may redistribute and modify this documentation under the terms of the CERN OHL v.1.2. (http://ohwr.org/cernohl). \nThis documentation is distributed WITHOUT ANY EXPRESS OR IMPLIED WARRANTY, INCLUDING OF MERCHANTABILITY, SATISFACTORY \nQUALITY AND FITNESS FOR A PARTICULAR PURPOSE. Please see the CERN OHL v.1.2  for applicable conditions
+JECCbot ECU
 Text Label 7900 3700 0    60   ~ 0
 INH12

Commit message: component placement almost done
Parts:
- removed X1: 8MHz, crystals:Crystal_HC49-U_Vertical, symbol devices:QUARTZCMS4
- added Y1: Crystal_Small, crystals:Crystal_HC49-U_Vertical, symbol devices:Crystal_Small
Connections:
- net OSC_IN: now also U1.5 (PD0/RCC_OSC_IN), Y1.1; no longer U1.3 (PC14/RCC_OSC32_IN)
- net OSC_OUT: now also U1.6 (PD1/RCC_OSC_OUT), Y1.2; no longer U1.4 (PC15/ADC1_EXTI15/ADC2_EXTI15/RCC_OSC32_OUT)
Changed lines of the file:
@@
 Text GLabel 8550 3300 2    60   Input ~ 0
 VIN_MEAS
-Text GLabel 1500 2900 0    60   Input ~ 0
+Text GLabel 1500 2500 0    60   Input ~ 0
 OSC_IN
 $Sheet
@@
 Wire Wire Line
 	10250 1100 10250 1000
-$Comp
-L devices:QUARTZCMS4 X1
-U 1 1 5E89B855
-P 10100 4000
-F 0 "X1" H 10100 4355 50  0000 C CNN
-F 1 "8MHz" H 10100 4264 50  0000 C CNN
-F 2 "crystals:Crystal_HC49-U_Vertical" H 10100 4173 50  0000 C CNN
-F 3 "" H 10100 4000 50  0000 C CNN
-	1    10100 4000
-	1    0    0    1
-$EndComp
 $Comp
 L devices:R_0603 R1
@@
 	10400 4750 10400 4650
 Wire Wire Line
-	10400 4450 10400 4000
-Wire Wire Line
-	9800 4000 9800 4450
-Wire Wire Line
-	9800 4000 9800 3550
-Wire Wire Line
 	9800 3550 10000 3550
-Connection ~ 9800 4000
 Wire Wire Line
 	10200 3550 10400 3550
-Wire Wire Line
-	10400 3550 10400 4000
-Connection ~ 10400 4000
 Wire Wire Line
 	10400 3350 10400 3550
@@
 	9800 3350 9800 3550
 Connection ~ 9800 3550
-Text GLabel 1500 3000 0    60   Output ~ 0
+Text GLabel 1500 2600 0    60   Output ~ 0
 OSC_OUT
 Text GLabel 9800 3350 1    50   Output ~ 0
@@
 NoConn ~ 7800 4000
 NoConn ~ 7800 4700
-NoConn ~ 2000 2500
-NoConn ~ 2000 2600
+NoConn ~ 2000 2900
+NoConn ~ 2000 3000
 NoConn ~ 2000 4100
 NoConn ~ 2000 4400
@@
 SPI_SCK
 Wire Wire Line
-	7800 3600 8450 3600
-Wire Wire Line
-	7800 3700 8450 3700
-Wire Wire Line
-	7800 3900 8450 3900
-Wire Wire Line
-	7800 3800 8450 3800
-Wire Wire Line
-	7800 3300 8550 3300
-Wire Wire Line
-	7800 4100 8450 4100
-Wire Wire Line
-	7800 4200 8450 4200
-Wire Wire Line
-	7800 4300 8450 4300
-Wire Wire Line
-	7800 4400 8450 4400
-Wire Wire Line
-	7800 3400 8450 3400
-Wire Wire Line
-	7800 3500 8450 3500
-Wire Wire Line
-	7800 4500 8450 4500
-Wire Wire Line
-	7800 4600 8450 4600
-Wire Wire Line
 	5000 5100 5000 5250
 Wire Wire Line
@@
 	1350 3400 2000 3400
 Wire Wire Line
-	1500 2900 2000 2900
-Wire Wire Line
-	1500 3000 2000 3000
+	1500 2500 2000 2500
+Wire Wire Line
+	1500 2600 2000 2600
 Wire Wire Line
 	1350 3500 2000 3500
@@
 GPIO
 Wire Wire Line
-	8450 3200 7800 3200
+	7800 3600 8450 3600
+Wire Wire Line
+	7800 3700 8450 3700
+Wire Wire Line
+	7800 3900 8450 3900
+Wire Wire Line
+	7800 3800 8450 3800
+Wire Wire Line
+	7800 3300 8550 3300
+Wire Wire Line
+	7800 4100 8450 4100
+Wire Wire Line
+	7800 4200 8450 4200
+Wire Wire Line
+	7800 4300 8450 4300
+Wire Wire Line
+	7800 4400 8450 4400
+Wire Wire Line
+	7800 3400 8450 3400
+Wire Wire Line
+	7800 3500 8450 3500
+Wire Wire Line
+	7800 4500 8450 4500
+Wire Wire Line
+	7800 4600 8450 4600
+Wire Wire Line
+	7800 3200 8450 3200
+Wire Wire Line
+	9800 3550 9800 4100
+Wire Wire Line
+	10400 3550 10400 4100
+$Comp
+L devices:Crystal_Small Y1
+U 1 1 5E8F0531
+P 10100 4100
+F 0 "Y1" H 10100 4415 50  0000 C CNN
+F 1 "Crystal_Small" H 10100 4324 50  0000 C CNN
+F 2 "crystals:Crystal_HC49-U_Vertical" H 10100 4233 50  0000 C CNN
+F 3 "" H 10100 4100 50  0000 C CNN
+	1    10100 4100
+	1    0    0    -1
+$EndComp
+Wire Wire Line
+	10200 4100 10400 4100
+Connection ~ 10400 4100
+Wire Wire Line
+	10400 4100 10400 4450
+Wire Wire Line
+	10000 4100 9800 4100
+Connection ~ 9800 4100
+Wire Wire Line
+	9800 4100 9800 4450
 $EndSCHEMATC

Commit message: updated schematics
Other:
- note removed: "JECCbot ECU"
Changed lines of the file:
@@
 encoding utf-8
 Sheet 1 5
-Title "HighPowerMotorFeatherWing"
+Title "JECCbotECU"
 Date "2019-12-29"
 Rev "1.0"
-Comp "generationmake"
+Comp "JECC"
 Comment1 ""
 Comment2 ""
 Comment3 ""
-Comment4 "This documentation describes Open Hardware and is licensed under the CERN OHL v. 1.2."
+Comment4 ""
 $EndDescr
-Text Notes 500  650  0    47   ~ 0
-JECCbot ECU
 Text Label 7900 3700 0    60   ~ 0
 INH12
