File: hardware/kicad/bno055.sch (KiCad schematic (older format))
At the start: 7 parts, among them U4 BNO055

Commit message: finished schematics
Parts:
- renumbered R9 to R12, R10 to R13
Changed lines of the file:
@@
 $EndComp
 $Comp
-L devices:R_0603 R9
+L devices:R_0603 R12
 U 1 1 5E9FF9B5
 P 3450 3500
-F 0 "R9" H 3509 3546 50  0000 L CNN
+F 0 "R12" H 3509 3546 50  0000 L CNN
 F 1 "10k" H 3509 3455 50  0000 L CNN
 F 2 "resistors:R_0603" H 3450 3350 50  0001 C CNN
@@
 $EndComp
 $Comp
-L devices:R_0603 R10
+L devices:R_0603 R13
 U 1 1 5E9FFB71
 P 3450 3400
-F 0 "R10" H 3509 3446 50  0000 L CNN
+F 0 "R13" H 3509 3446 50  0000 L CNN
 F 1 "10k" H 3509 3355 50  0000 L CNN
 F 2 "resistors:R_0603" H 3450 3250 50  0001 C CNN
@@
 	3900 4300 3700 4300
 $Comp
-L power-supply:GND #PWR?
+L power-supply:GND #PWR0143
 U 1 1 5EA2B085
 P 5800 3400
-F 0 "#PWR?" H 5800 3150 50  0001 C CNN
+F 0 "#PWR0143" H 5800 3150 50  0001 C CNN
 F 1 "GND" V 5805 3272 50  0000 R CNN
 F 2 "" H 5800 3400 50  0000 C CNN
@@
 $EndComp
 $Comp
-L power-supply:GND #PWR?
+L power-supply:GND #PWR0144
 U 1 1 5EA2B2E3
 P 3100 3700
-F 0 "#PWR?" H 3100 3450 50  0001 C CNN
+F 0 "#PWR0144" H 3100 3450 50  0001 C CNN
 F 1 "GND" V 3105 3572 50  0000 R CNN
 F 2 "" H 3100 3700 50  0000 C CNN
@@
 	3700 4200 3700 4300
 $Comp
-L power-supply:GND #PWR?
+L power-supply:GND #PWR0145
 U 1 1 5EA2BC43
 P 5800 4300
-F 0 "#PWR?" H 5800 4050 50  0001 C CNN
+F 0 "#PWR0145" H 5800 4050 50  0001 C CNN
 F 1 "GND" V 5805 4172 50  0000 R CNN
 F 2 "" H 5800 4300 50  0000 C CNN
@@
 	3700 4400 3700 4300
 $Comp
-L power-supply:GND #PWR?
+L power-supply:GND #PWR0146
 U 1 1 5EA2C40F
 P 3700 4650
-F 0 "#PWR?" H 3700 4400 50  0001 C CNN
+F 0 "#PWR0146" H 3700 4400 50  0001 C CNN
 F 1 "GND" H 3705 4477 50  0000 C CNN
 F 2 "" H 3700 4650 50  0000 C CNN
@@
 	3750 2650 3900 2650
 $Comp
-L power-supply:+3V3 #PWR?
+L power-supply:+3V3 #PWR0147
 U 1 1 5EA2FED4
 P 3750 2250
-F 0 "#PWR?" H 3750 2100 50  0001 C CNN
+F 0 "#PWR0147" H 3750 2100 50  0001 C CNN
 F 1 "+3V3" H 3765 2423 50  0000 C CNN
 F 2 "" H 3750 2250 50  0000 C CNN
@@
 	3250 2550 3350 2550
 $Comp
-L power-supply:GND #PWR?
+L power-supply:GND #PWR0148
 U 1 1 5EA31EA0
 P 3100 2750
-F 0 "#PWR?" H 3100 2500 50  0001 C CNN
+F 0 "#PWR0148" H 3100 2500 50  0001 C CNN
 F 1 "GND" V 3105 2622 50  0000 R CNN
 F 2 "" H 3100 2750 50  0000 C CNN
@@
 	3250 3400 3350 3400
 $Comp
-L power-supply:+3V3 #PWR?
+L power-supply:+3V3 #PWR0149
 U 1 1 5EA33ECD
 P 3050 3400
-F 0 "#PWR?" H 3050 3250 50  0001 C CNN
+F 0 "#PWR0149" H 3050 3250 50  0001 C CNN
 F 1 "+3V3" V 3065 3528 50  0000 L CNN
 F 2 "" H 3050 3400 50  0000 C CNN
@@
 NoConn ~ 5400 3750
 $Comp
-L power-supply:+3V3 #PWR?
+L power-supply:+3V3 #PWR0150
 U 1 1 5EA3558F
 P 3050 4300
-F 0 "#PWR?" H 3050 4150 50  0001 C CNN
+F 0 "#PWR0150" H 3050 4150 50  0001 C CNN
 F 1 "+3V3" V 3065 4428 50  0000 L CNN
 F 2 "" H 3050 4300 50  0000 C CNN

Commit message: finished layout
Parts:
- added R20, R21: 10k, resistors:R_0603, symbol devices:R_0603
Connections:
- net +3V3: now also R20.1, R21.1
- net I2C_SCL: now also R21.2
- net I2C_SDA: now also R20.2
Changed lines of the file:
@@
 Wire Wire Line
 	3350 4300 3050 4300
-Text GLabel 5600 4100 2    50   BiDi ~ 0
+Text GLabel 6600 4100 2    50   BiDi ~ 0
 I2C_SDA
-Text GLabel 5600 4200 2    50   Input ~ 0
+Text GLabel 6600 4200 2    50   Input ~ 0
 I2C_SCL
 Wire Wire Line
-	5600 4100 5400 4100
+	5400 4100 5850 4100
 Wire Wire Line
-	5400 4200 5600 4200
+	5400 4200 6400 4200
+$Comp
+L devices:R_0603 R20
+U 1 1 5E97804D
+P 5850 3850
+F 0 "R20" H 5909 3896 50  0000 L CNN
+F 1 "10k" H 5909 3805 50  0000 L CNN
+F 2 "resistors:R_0603" H 5850 3700 50  0001 C CNN
+F 3 "" H 5850 3850 50  0000 C CNN
+	1    5850 3850
+	1    0    0    -1
+$EndComp
+$Comp
+L devices:R_0603 R21
+U 1 1 5E9781BC
+P 6400 3850
+F 0 "R21" H 6459 3896 50  0000 L CNN
+F 1 "10k" H 6459 3805 50  0000 L CNN
+F 2 "resistors:R_0603" H 6400 3700 50  0001 C CNN
+F 3 "" H 6400 3850 50  0000 C CNN
+	1    6400 3850
+	1    0    0    -1
+$EndComp
+Wire Wire Line
+	5850 4100 5850 3950
+Connection ~ 5850 4100
+Wire Wire Line
+	5850 4100 6600 4100
+Wire Wire Line
+	6400 3950 6400 4200
+Connection ~ 6400 4200
+Wire Wire Line
+	6400 4200 6600 4200
+Wire Wire Line
+	5850 3750 5850 3650
+Wire Wire Line
+	5850 3650 6400 3650
+Wire Wire Line
+	6400 3650 6400 3750
+$Comp
+L power-supply:+3V3 #PWR?
+U 1 1 5E97B2A1
+P 6400 3500
+F 0 "#PWR?" H 6400 3350 50  0001 C CNN
+F 1 "+3V3" H 6415 3673 50  0000 C CNN
+F 2 "" H 6400 3500 50  0000 C CNN
+F 3 "" H 6400 3500 50  0000 C CNN
+	1    6400 3500
+	1    0    0    -1
+$EndComp
+Wire Wire Line
+	6400 3500 6400 3650
+Connection ~ 6400 3650
 $EndSCHEMATC
