File: hardware/kicad/connectors.sch (KiCad schematic (older format))
At the start: 18 parts, among them CN2 691382010004, CN2 691382010005, CN3 691382010004, P1 USB_B, P2 CONN_02X05, P3 CONN_02X03, U2 BSS138, U3 BSS138

Commit message: bugfix
Connections:
- net +5V: now also R8.1; no longer R8.2
- net KVH_RX: now also R7.2, R9.2, U2.3; no longer R10.2, R11.1
- net KVH_TX: now also R10.1, U3.1; no longer R8.1, R9.1, U3.3
- net at U2.1: now also CN2.3 (P3), R11.1, R9.1
- new net: CN2.2 (P2), R10.2, R8.2, U3.3
Other:
- moved on the sheet: CN2, P2, R10, R11, R4, R7, R8, R9, U2, U3

Commit message: finished schematics
Parts:
- added P4: CONN_02X05, pin_headers:Pin_Header_Angled_2x05, symbol mechanical-connectors:CONN_02X05
- renumbered CN2 to CN3, CN3 to CN4
Connections:
- net +12V: now also P4.3 (P3)
- net +3V3: now also P4.7 (P7)
- net +5V: now also P4.5 (P5)
- net GND: now also P4.1 (P1)
- new net GPIO: P4.9 (P9)
- new net I2C_SCL: P4.2 (P2)
- new net I2C_SDA: P4.4 (P4)
- new net SPI_MISO: P4.8 (P8)
- new net SPI_MOSI: P4.10 (P10)
- new net SPI_SCK: P4.6 (P6)
Changed lines of the file:
@@
 KVH_RX
 $Comp
-L CON_wuerth:691382010005 CN2
+L CON_wuerth:691382010005 CN3
 U 1 1 5E978D9C
 P 5250 2650
-F 0 "CN2" H 5167 2135 50  0000 C CNN
+F 0 "CN3" H 5167 2135 50  0000 C CNN
 F 1 "691382010005" H 5167 2226 50  0000 C CNN
 F 2 "CON_wuerth:WR-TBL_691382010005" H 5167 2317 50  0000 C CNN
@@
 $EndComp
 $Comp
-L power-supply:+5V #PWR?
+L power-supply:+5V #PWR0126
 U 1 1 5E97A28C
 P 6150 2300
-F 0 "#PWR?" H 6150 2150 50  0001 C CNN
+F 0 "#PWR0126" H 6150 2150 50  0001 C CNN
 F 1 "+5V" V 6165 2428 50  0000 L CNN
 F 2 "" H 6150 2300 50  0000 C CNN
@@
 $EndComp
 $Comp
-L power-supply:GND #PWR?
+L power-supply:GND #PWR0127
 U 1 1 5E97A88E
 P 6850 3000
-F 0 "#PWR?" H 6850 2750 50  0001 C CNN
+F 0 "#PWR0127" H 6850 2750 50  0001 C CNN
 F 1 "GND" V 6855 2872 50  0000 R CNN
 F 2 "" H 6850 3000 50  0000 C CNN
@@
 	5450 2450 6150 2450
 $Comp
-L CON_wuerth:691382010004 CN3
+L CON_wuerth:691382010004 CN4
 U 1 1 5E985ABB
 P 7900 2700
-F 0 "CN3" H 7817 2235 50  0000 C CNN
+F 0 "CN4" H 7817 2235 50  0000 C CNN
 F 1 "691382010004" H 7817 2326 50  0000 C CNN
 F 2 "CON_wuerth:WR-TBL_691382010004" H 7817 2417 50  0000 C CNN
@@
 $EndComp
 $Comp
-L power-supply:+3V3 #PWR?
+L power-supply:+3V3 #PWR0128
 U 1 1 5E98AFDC
 P 8750 2550
-F 0 "#PWR?" H 8750 2400 50  0001 C CNN
+F 0 "#PWR0128" H 8750 2400 50  0001 C CNN
 F 1 "+3V3" V 8765 2678 50  0000 L CNN
 F 2 "" H 8750 2550 50  0000 C CNN
@@
 $EndComp
 $Comp
-L power-supply:GND #PWR?
+L power-supply:GND #PWR0129
 U 1 1 5E98B42F
 P 8750 2850
-F 0 "#PWR?" H 8750 2600 50  0001 C CNN
+F 0 "#PWR0129" H 8750 2600 50  0001 C CNN
 F 1 "GND" V 8755 2722 50  0000 R CNN
 F 2 "" H 8750 2850 50  0000 C CNN
@@
 	2000 4200 2000 4100
 $Comp
-L power-supply:GND #PWR?
+L power-supply:GND #PWR0130
 U 1 1 5EA310DC
 P 2000 4950
-F 0 "#PWR?" H 2000 4700 50  0001 C CNN
+F 0 "#PWR0130" H 2000 4700 50  0001 C CNN
 F 1 "GND" H 2005 4777 50  0000 C CNN
 F 2 "" H 2000 4950 50  0000 C CNN
@@
 Wire Wire Line
 	3150 2750 3750 2750
+$Comp
+L mechanical-connectors:CONN_02X05 P4
+U 1 1 5E8AD3DA
+P 5750 4750
+F 0 "P4" H 5750 5255 50  0000 C CNN
+F 1 "CONN_02X05" H 5750 5164 50  0000 C CNN
+F 2 "pin_headers:Pin_Header_Angled_2x05" H 5750 5073 50  0000 C CNN
+F 3 "" H 5750 3550 50  0000 C CNN
+	1    5750 4750
+	1    0    0    1
+$EndComp
+$Comp
+L power-supply:GND #PWR?
+U 1 1 5E8C8A73
+P 4700 5150
+F 0 "#PWR?" H 4700 4900 50  0001 C CNN
+F 1 "GND" H 4705 4977 50  0000 C CNN
+F 2 "" H 4700 5150 50  0000 C CNN
+F 3 "" H 4700 5150 50  0000 C CNN
+	1    4700 5150
+	1    0    0    -1
+$EndComp
+$Comp
+L power-supply:+3V3 #PWR?
+U 1 1 5E8C9187
+P 4700 4400
+F 0 "#PWR?" H 4700 4250 50  0001 C CNN
+F 1 "+3V3" H 4715 4573 50  0000 C CNN
+F 2 "" H 4700 4400 50  0000 C CNN
+F 3 "" H 4700 4400 50  0000 C CNN
+	1    4700 4400
+	1    0    0    -1
+$EndComp
+$Comp
+L power-supply:+5V #PWR?
+U 1 1 5E8C9724
+P 4450 4400
+F 0 "#PWR?" H 4450 4250 50  0001 C CNN
+F 1 "+5V" H 4465 4573 50  0000 C CNN
+F 2 "" H 4450 4400 50  0000 C CNN
+F 3 "" H 4450 4400 50  0000 C CNN
+	1    4450 4400
+	1    0    0    -1
+$EndComp
+$Comp
+L power-supply:+12V #PWR?
+U 1 1 5E8C9D3E
+P 4200 4400
+F 0 "#PWR?" H 4200 4250 50  0001 C CNN
+F 1 "+12V" H 4215 4573 50  0000 C CNN
+F 2 "" H 4200 4400 50  0000 C CNN
+F 3 "" H 4200 4400 50  0000 C CNN
+	1    4200 4400
+	1    0    0    -1
+$EndComp
+Wire Wire Line
+	5500 4950 4700 4950
+Wire Wire Line
+	4700 4950 4700 5150
+Wire Wire Line
+	5500 4850 4200 4850
+Wire Wire Line
+	4200 4850 4200 4400
+Wire Wire Line
+	5500 4750 4450 4750
+Wire Wire Line
+	4450 4750 4450 4400
+Wire Wire Line
+	5500 4650 4700 4650
+Wire Wire Line
+	4700 4650 4700 4400
+Text GLabel 6400 4950 2    50   Input ~ 0
+I2C_SCL
+Text GLabel 6400 4850 2    50   BiDi ~ 0
+I2C_SDA
+Wire Wire Line
+	6400 4950 6000 4950
+Wire Wire Line
+	6000 4850 6400 4850
+Text GLabel 5200 4550 0    50   BiDi ~ 0
+GPIO
+Text GLabel 6400 4750 2    50   Input ~ 0
+SPI_SCK
+Text GLabel 6400 4550 2    50   Input ~ 0
+SPI_MOSI
+Text GLabel 6400 4650 2    50   Output ~ 0
+SPI_MISO
+Wire Wire Line
+	5500 4550 5200 4550
+Wire Wire Line
+	6000 4550 6400 4550
+Wire Wire Line
+	6000 4650 6400 4650
+Wire Wire Line
+	6400 4750 6000 4750
 $EndSCHEMATC

Commit message: finished layout
Parts:
- added P5: WR-TBL_691313710002, mechanical-connectors:WR-TBL_691313710002, symbol mechanical-connectors:WR-TBL_691313710002
Connections:
- new net VBAT: P5.1 (P1)
Changed lines of the file:
@@
 Wire Wire Line
 	6400 4750 6000 4750
+$Comp
+L mechanical-connectors:WR-TBL_691313710002 P5
+U 1 1 5E98B38F
+P 9550 4650
+F 0 "P5" H 9628 4691 50  0000 L CNN
+F 1 "WR-TBL_691313710002" H 9628 4600 50  0000 L CNN
+F 2 "mechanical-connectors:WR-TBL_691313710002" H 9450 4700 50  0001 C CNN
+F 3 "" H 9550 4650 50  0000 C CNN
+	1    9550 4650
+	1    0    0    -1
+$EndComp
+$Comp
+L power-supply:GND #PWR?
+U 1 1 5E98D818
+P 8750 4900
+F 0 "#PWR?" H 8750 4650 50  0001 C CNN
+F 1 "GND" H 8755 4727 50  0000 C CNN
+F 2 "" H 8750 4900 50  0000 C CNN
+F 3 "" H 8750 4900 50  0000 C CNN
+	1    8750 4900
+	1    0    0    -1
+$EndComp
+Text GLabel 8750 4600 0    50   Output ~ 0
+VBAT
+Wire Wire Line
+	8750 4600 9350 4600
+Wire Wire Line
+	9300 4700 8750 4700
+Wire Wire Line
+	8750 4700 8750 4900
 $EndSCHEMATC

Commit message: design rules check
Parts:
- renumbered P5 to BAT1, P3 to Boot1, CN2 to Compass1, P2 to Debug1, P4 to GPIO1, CN4 to GPS1, CN3 to Lidar1
Changed lines of the file:
@@
 $EndComp
 $Comp
-L mechanical-connectors:CONN_02X05 P2
+L mechanical-connectors:CONN_02X05 Debug1
 U 1 1 5E8E0B26
 P 4050 1200
-F 0 "P2" H 4050 1705 50  0000 C CNN
+F 0 "Debug1" H 4050 1705 50  0000 C CNN
 F 1 "CONN_02X05" H 4050 1614 50  0000 C CNN
 F 2 "pin_headers:Pin_Header_Angled_2x05" H 4050 1523 50  0000 C CNN
@@
 NoConn ~ 3800 1400
 $Comp
-L mechanical-connectors:CONN_02X03 P3
+L mechanical-connectors:CONN_02X03 Boot1
 U 1 1 5E8EA477
 P 6950 1300
-F 0 "P3" H 6950 1705 50  0000 C CNN
+F 0 "Boot1" H 6950 1705 50  0000 C CNN
 F 1 "CONN_02X03" H 6950 1614 50  0000 C CNN
 F 2 "pin_headers:Pin_Header_Angled_2x03" H 6950 1523 50  0000 C CNN
@@
 	6350 1300 6250 1300
 $Comp
-L CON_wuerth:691382010004 CN2
+L CON_wuerth:691382010004 Compass1
 U 1 1 5E8F806A
 P 3950 2700
-F 0 "CN2" H 3867 2235 50  0000 C CNN
+F 0 "Compass1" H 3867 2235 50  0000 C CNN
 F 1 "691382010004" H 3867 2326 50  0000 C CNN
 F 2 "CON_wuerth:WR-TBL_691382010004" H 3867 2417 50  0000 C CNN
@@
 KVH_RX
 $Comp
-L CON_wuerth:691382010005 CN3
+L CON_wuerth:691382010005 Lidar1
 U 1 1 5E978D9C
 P 5250 2650
-F 0 "CN3" H 5167 2135 50  0000 C CNN
+F 0 "Lidar1" H 5167 2135 50  0000 C CNN
 F 1 "691382010005" H 5167 2226 50  0000 C CNN
 F 2 "CON_wuerth:WR-TBL_691382010005" H 5167 2317 50  0000 C CNN
@@
 	5450 2450 6150 2450
 $Comp
-L CON_wuerth:691382010004 CN4
+L CON_wuerth:691382010004 GPS1
 U 1 1 5E985ABB
 P 7900 2700
-F 0 "CN4" H 7817 2235 50  0000 C CNN
+F 0 "GPS1" H 7817 2235 50  0000 C CNN
 F 1 "691382010004" H 7817 2326 50  0000 C CNN
 F 2 "CON_wuerth:WR-TBL_691382010004" H 7817 2417 50  0000 C CNN
@@
 	3150 2750 3750 2750
 $Comp
-L mechanical-connectors:CONN_02X05 P4
+L mechanical-connectors:CONN_02X05 GPIO1
 U 1 1 5E8AD3DA
 P 5750 4750
-F 0 "P4" H 5750 5255 50  0000 C CNN
+F 0 "GPIO1" H 5750 5255 50  0000 C CNN
 F 1 "CONN_02X05" H 5750 5164 50  0000 C CNN
 F 2 "pin_headers:Pin_Header_Angled_2x05" H 5750 5073 50  0000 C CNN
@@
 $EndComp
 $Comp
-L power-supply:GND #PWR?
+L power-supply:GND #PWR0134
 U 1 1 5E8C8A73
 P 4700 5150
-F 0 "#PWR?" H 4700 4900 50  0001 C CNN
+F 0 "#PWR0134" H 4700 4900 50  0001 C CNN
 F 1 "GND" H 4705 4977 50  0000 C CNN
 F 2 "" H 4700 5150 50  0000 C CNN
@@
 $EndComp
 $Comp
-L power-supply:+3V3 #PWR?
+L power-supply:+3V3 #PWR0151
 U 1 1 5E8C9187
 P 4700 4400
-F 0 "#PWR?" H 4700 4250 50  0001 C CNN
+F 0 "#PWR0151" H 4700 4250 50  0001 C CNN
 F 1 "+3V3" H 4715 4573 50  0000 C CNN
 F 2 "" H 4700 4400 50  0000 C CNN
@@
 $EndComp
 $Comp
-L power-supply:+5V #PWR?
+L power-supply:+5V #PWR0152
 U 1 1 5E8C9724
 P 4450 4400
-F 0 "#PWR?" H 4450 4250 50  0001 C CNN
+F 0 "#PWR0152" H 4450 4250 50  0001 C CNN
 F 1 "+5V" H 4465 4573 50  0000 C CNN
 F 2 "" H 4450 4400 50  0000 C CNN
@@
 $EndComp
 $Comp
-L power-supply:+12V #PWR?
+L power-supply:+12V #PWR0153
 U 1 1 5E8C9D3E
 P 4200 4400
-F 0 "#PWR?" H 4200 4250 50  0001 C CNN
+F 0 "#PWR0153" H 4200 4250 50  0001 C CNN
 F 1 "+12V" H 4215 4573 50  0000 C CNN
 F 2 "" H 4200 4400 50  0000 C CNN
@@
 	6400 4750 6000 4750
 $Comp
-L mechanical-connectors:WR-TBL_691313710002 P5
+L mechanical-connectors:WR-TBL_691313710002 BAT1
 U 1 1 5E98B38F
 P 9550 4650
-F 0 "P5" H 9628 4691 50  0000 L CNN
+F 0 "BAT1" H 9628 4691 50  0000 L CNN
 F 1 "WR-TBL_691313710002" H 9628 4600 50  0000 L CNN
 F 2 "mechanical-connectors:WR-TBL_691313710002" H 9450 4700 50  0001 C CNN
@@
 $EndComp
 $Comp
-L power-supply:GND #PWR?
+L power-supply:GND #PWR0154
 U 1 1 5E98D818
 P 8750 4900
-F 0 "#PWR?" H 8750 4650 50  0001 C CNN
+F 0 "#PWR0154" H 8750 4650 50  0001 C CNN
 F 1 "GND" H 8755 4727 50  0000 C CNN
 F 2 "" H 8750 4900 50  0000 C CNN
