File: hardware/kicad/power.sch (KiCad schematic (older format))
At the start: 24 parts

Commit message: finished schematics
Parts:
- gave numbers to parts that had none: 24
Changed lines of the file:
@@
 $EndDescr
 $Comp
-L voltage-regulators:GAPTEC_6S8W4_1.6RP U?
+L voltage-regulators:GAPTEC_6S8W4_1.6RP U6
 U 1 1 5E3D4DCC
 P 6050 1300
-F 0 "U?" H 6050 1675 50  0000 C CNN
+F 0 "U6" H 6050 1675 50  0000 C CNN
 F 1 "GAPTEC_6S8W4_1.6RP" H 6050 1584 50  0000 C CNN
 F 2 "MODULE_power:GAPTEC_6S8W4_1.6RP" H 6050 1700 50  0001 C CNN
@@
 $EndComp
 $Comp
-L devices:R_0603 R?
+L devices:R_0603 R16
 U 1 1 5E3D5A97
 P 5150 1100
-F 0 "R?" H 5209 1146 50  0000 L CNN
+F 0 "R16" H 5209 1146 50  0000 L CNN
 F 1 "DNI" H 5209 1055 50  0000 L CNN
 F 2 "resistors:R_0603" H 5150 950 50  0001 C CNN
@@
 $EndComp
 $Comp
-L devices:R_0603 R?
+L devices:R_0603 R17
 U 1 1 5E3D5C8F
 P 5150 1400
-F 0 "R?" H 5209 1446 50  0000 L CNN
+F 0 "R17" H 5209 1446 50  0000 L CNN
 F 1 "DNI" H 5209 1355 50  0000 L CNN
 F 2 "resistors:R_0603" H 5150 1250 50  0001 C CNN
@@
 	4950 950  4950 1200
 $Comp
-L devices:C_1210 C?
+L devices:C_1210 C16
 U 1 1 5E40C2CF
 P 4800 1350
-F 0 "C?" H 4892 1396 50  0000 L CNN
+F 0 "C16" H 4892 1396 50  0000 L CNN
 F 1 "4.7uF 50V" H 4550 1600 50  0000 L CNN
 F 2 "capacitors:C_1210" H 4800 1200 50  0001 C CNN
@@
 Connection ~ 4800 1200
 $Comp
-L devices:D_Small D?
+L devices:D_Small D1
 U 1 1 5E411723
 P 3350 1200
-F 0 "D?" H 3350 995 50  0000 C CNN
+F 0 "D1" H 3350 995 50  0000 C CNN
 F 1 "D_Small" H 3350 1086 50  0000 C CNN
 F 2 "diodes:SOD-123" H 3350 1087 50  0001 C CNN
@@
 	7000 1450 7000 1650
 $Comp
-L power-supply:GND #PWR?
+L power-supply:GND #PWR0131
 U 1 1 5E413C27
 P 7000 1650
-F 0 "#PWR?" H 7000 1400 50  0001 C CNN
+F 0 "#PWR0131" H 7000 1400 50  0001 C CNN
 F 1 "GND" H 7005 1477 50  0000 C CNN
 F 2 "" H 7000 1650 50  0000 C CNN
@@
 	6450 1450 6600 1450
 $Comp
-L power-supply:+12V #PWR?
+L power-supply:+12V #PWR0132
 U 1 1 5E4147CA
 P 7000 900
-F 0 "#PWR?" H 7000 750 50  0001 C CNN
+F 0 "#PWR0132" H 7000 750 50  0001 C CNN
 F 1 "+12V" H 7015 1073 50  0000 C CNN
 F 2 "" H 7000 900 50  0000 C CNN
@@
 $EndComp
 $Comp
-L devices:C_1206 C?
+L devices:C_1206 C22
 U 1 1 5E414C85
 P 7000 1300
-F 0 "C?" H 7000 1400 50  0000 L CNN
+F 0 "C22" H 7000 1400 50  0000 L CNN
 F 1 "22uF" H 7100 1250 50  0000 L CNN
 F 2 "capacitors:C_1206" H 7000 1150 50  0001 C CNN
@@
 $EndComp
 $Comp
-L devices:C_1206 C?
+L devices:C_1206 C20
 U 1 1 5E414FEF
 P 6800 1300
-F 0 "C?" H 6800 1400 50  0000 L CNN
+F 0 "C20" H 6800 1400 50  0000 L CNN
 F 1 "22uF" H 7100 1250 50  0000 L CNN
 F 2 "capacitors:C_1206" H 6800 1150 50  0001 C CNN
@@
 $EndComp
 $Comp
-L devices:C_1206 C?
+L devices:C_1206 C19
 U 1 1 5E4151CA
 P 6600 1300
-F 0 "C?" H 6600 1400 50  0000 L CNN
+F 0 "C19" H 6600 1400 50  0000 L CNN
 F 1 "22uF" H 7100 1250 50  0000 L CNN
 F 2 "capacitors:C_1206" H 6600 1150 50  0001 C CNN
@@
 	6600 1150 6800 1150
 $Comp
-L voltage-regulators:TPS54335A U?
+L voltage-regulators:TPS54335A U5
 U 1 1 5E4197F3
 P 4850 3350
-F 0 "U?" H 4850 4190 50  0000 C CNN
+F 0 "U5" H 4850 4190 50  0000 C CNN
 F 1 "TPS54335A" H 4850 4099 50  0000 C CNN
 F 2 "SOIC:SOIC-8-1EP_3.9x4.9mm_Pitch1.27mm" H 4750 3250 50  0001 C CNN
@@
 	4000 3850 4000 4000
 $Comp
-L power-supply:GND #PWR?
+L power-supply:GND #PWR0133
 U 1 1 5E4202CE
 P 4000 4050
-F 0 "#PWR?" H 4000 3800 50  0001 C CNN
+F 0 "#PWR0133" H 4000 3800 50  0001 C CNN
 F 1 "GND" H 4005 3877 50  0000 C CNN
 F 2 "" H 4000 4050 50  0000 C CNN
@@
 	4000 2850 4000 2750
 $Comp
-L power-supply:+12V #PWR?
+L power-supply:+12V #PWR0134
 U 1 1 5E4230DE
 P 4000 2600
-F 0 "#PWR?" H 4000 2450 50  0001 C CNN
+F 0 "#PWR0134" H 4000 2450 50  0001 C CNN
 F 1 "+12V" H 4015 2773 50  0000 C CNN
 F 2 "" H 4000 2600 50  0000 C CNN
@@
 	2500 3300 2500 3450
 $Comp
-L devices:R_0603 R?
+L devices:R_0603 R14
 U 1 1 5E425834
 P 2500 3550
-F 0 "R?" H 2559 3596 50  0000 L CNN
+F 0 "R14" H 2559 3596 50  0000 L CNN
 F 1 "143k" H 2559 3505 50  0000 L CNN
 F 2 "resistors:R_0603" H 2500 3400 50  0001 C CNN
@@
 $EndComp
 $Comp
-L power-supply:GND #PWR?
+L power-supply:GND #PWR0135
 U 1 1 5E426935
 P 2500 3800
-F 0 "#PWR?" H 2500 3550 50  0001 C CNN
+F 0 "#PWR0135" H 2500 3550 50  0001 C CNN
 F 1 "GND" H 2505 3627 50  0000 C CNN
 F 2 "" H 2500 3800 50  0000 C CNN
@@
 	3450 3900 3450 4250
 $Comp
-L devices:R_0603 R?
+L devices:R_0603 R15
 U 1 1 5E4296CE
 P 3450 4350
-F 0 "R?" H 3509 4396 50  0000 L CNN
+F 0 "R15" H 3509 4396 50  0000 L CNN
 F 1 "3.74k" H 3509 4305 50  0000 L CNN
 F 2 "resistors:R_0603" H 3450 4200 50  0001 C CNN
@@
 $EndComp
 $Comp
-L power-supply:GND #PWR?
+L power-supply:GND #PWR0136
 U 1 1 5E4296D4
 P 3450 4550
-F 0 "#PWR?" H 3450 4300 50  0001 C CNN
+F 0 "#PWR0136" H 3450 4300 50  0001 C CNN
 F 1 "GND" H 3455 4377 50  0000 C CNN
 F 2 "" H 3450 4550 50  0000 C CNN
@@
 	3450 4450 3450 4500
 $Comp
-L devices:C_0603 C?
+L devices:C_0603 C13
 U 1 1 5E42A6E4
 P 3450 3800
-F 0 "C?" H 3542 3846 50  0000 L CNN
+F 0 "C13" H 3542 3846 50  0000 L CNN
 F 1 "12n" H 3542 3755 50  0000 L CNN
 F 2 "capacitors:C_0603" H 3450 3650 50  0001 C CNN
@@
 $EndComp
 $Comp
-L devices:C_0603 C?
+L devices:C_0603 C11
 U 1 1 5E42AB7F
 P 3000 3950
-F 0 "C?" H 3092 3996 50  0000 L CNN
+F 0 "C11" H 3092 3996 50  0000 L CNN
 F 1 "120p" H 3092 3905 50  0000 L CNN
 F 2 "capacitors:C_0603" H 3000 3800 50  0001 C CNN
@@
 	3450 3500 4100 3500
 $Comp
-L devices:R_0603 R?
+L devices:R_0603 R18
 U 1 1 5E439932
 P 7650 3550
-F 0 "R?" H 7709 3596 50  0000 L CNN
+F 0 "R18" H 7709 3596 50  0000 L CNN
 F 1 "100k" H 7709 3505 50  0000 L CNN
 F 2 "resistors:R_0603" H 7650 3400 50  0001 C CNN
@@
 $EndComp
 $Comp
-L devices:R_0603 R?
+L devices:R_0603 R19
 U 1 1 5E43A340
 P 7650 3950
-F 0 "R?" H 7709 3996 50  0000 L CNN
+F 0 "R19" H 7709 3996 50  0000 L CNN
 F 1 "19.1k" H 7709 3905 50  0000 L CNN
 F 2 "resistors:R_0603" H 7650 3800 50  0001 C CNN
@@
 	7650 4050 7650 4200
 $Comp
-L power-supply:GND #PWR?
+L power-supply:GND #PWR0137
 U 1 1 5E43F02B
 P 7650 4200
-F 0 "#PWR?" H 7650 3950 50  0001 C CNN
+F 0 "#PWR0137" H 7650 3950 50  0001 C CNN
 F 1 "GND" H 7655 4027 50  0000 C CNN
 F 2 "" H 7650 4200 50  0000 C CNN
@@
 $EndComp
 $Comp
-L devices:C_0603 C?
+L devices:C_0603 C17
 U 1 1 5E43F2C2
 P 5800 2850
-F 0 "C?" V 5571 2850 50  0000 C CNN
+F 0 "C17" V 5571 2850 50  0000 C CNN
 F 1 "100n" V 5662 2850 50  0000 C CNN
 F 2 "capacitors:C_0603" H 5800 2700 50  0001 C CNN
@@
 Connection ~ 6100 3250
 $Comp
-L devices:INDUCTOR_SMALL L?
+L devices:INDUCTOR_SMALL L2
 U 1 1 5E44A1D0
 P 6600 3250
-F 0 "L?" H 6600 3465 50  0000 C CNN
+F 0 "L2" H 6600 3465 50  0000 C CNN
 F 1 "WE-74437324150" H 6600 3374 50  0000 C CNN
 F 2 "L_power:WE-LHMI40xx" H 6600 3373 50  0001 C CNN
@@
 	6850 3250 6900 3250
 $Comp
-L devices:C_1206 C?
+L devices:C_1206 C21
 U 1 1 5E457184
 P 6900 3400
-F 0 "C?" H 6992 3446 50  0000 L CNN
+F 0 "C21" H 6992 3446 50  0000 L CNN
 F 1 "22u" H 7200 3350 50  0000 L CNN
 F 2 "capacitors:C_1206" H 6900 3250 50  0001 C CNN
@@
 $EndComp
 $Comp
-L devices:C_1206 C?
+L devices:C_1206 C23
 U 1 1 5E457C29
 P 7100 3400
-F 0 "C?" H 7192 3446 50  0000 L CNN
+F 0 "C23" H 7192 3446 50  0000 L CNN
 F 1 "22u" H 7200 3350 50  0000 L CNN
 F 2 "capacitors:C_1206" H 7100 3250 50  0001 C CNN
@@
 	7100 3250 7100 3300
 $Comp
-L power-supply:GND #PWR?
+L power-supply:GND #PWR0138
 U 1 1 5E45D25B
 P 7100 3550
-F 0 "#PWR?" H 7100 3300 50  0001 C CNN
+F 0 "#PWR0138" H 7100 3300 50  0001 C CNN
 F 1 "GND" H 7105 3377 50  0000 C CNN
 F 2 "" H 7100 3550 50  0000 C CNN
@@
 $EndComp
 $Comp
-L power-supply:GND #PWR?
+L power-supply:GND #PWR0139
 U 1 1 5E45EA0B
 P 6900 3550
-F 0 "#PWR?" H 6900 3300 50  0001 C CNN
+F 0 "#PWR0139" H 6900 3300 50  0001 C CNN
 F 1 "GND" H 6905 3377 50  0000 C CNN
 F 2 "" H 6900 3550 50  0000 C CNN
@@
 	7650 3750 7650 3850
 $Comp
-L power-supply:+5V #PWR?
+L power-supply:+5V #PWR0140
 U 1 1 5E478101
 P 7650 3050
-F 0 "#PWR?" H 7650 2900 50  0001 C CNN
+F 0 "#PWR0140" H 7650 2900 50  0001 C CNN
 F 1 "+5V" H 7665 3223 50  0000 C CNN
 F 2 "" H 7650 3050 50  0000 C CNN
@@
 Connection ~ 7650 3250
 $Comp
-L devices:C_1206 C?
+L devices:C_1206 C14
 U 1 1 5E47B024
 P 3550 2950
-F 0 "C?" H 3642 2996 50  0000 L CNN
+F 0 "C14" H 3642 2996 50  0000 L CNN
 F 1 "C_1206" H 3650 2900 50  0000 L CNN
 F 2 "capacitors:C_1206" H 3550 2800 50  0001 C CNN
@@
 $EndComp
 $Comp
-L devices:C_1206 C?
+L devices:C_1206 C12
 U 1 1 5E47BD2B
 P 3400 2950
-F 0 "C?" H 3492 2996 50  0000 L CNN
+F 0 "C12" H 3492 2996 50  0000 L CNN
 F 1 "C_1206" H 3650 2900 50  0000 L CNN
 F 2 "capacitors:C_1206" H 3400 2800 50  0001 C CNN
@@
 $EndComp
 $Comp
-L power-supply:GND #PWR?
+L power-supply:GND #PWR0141
 U 1 1 5E47D847
 P 3550 3100
-F 0 "#PWR?" H 3550 2850 50  0001 C CNN
+F 0 "#PWR0141" H 3550 2850 50  0001 C CNN
 F 1 "GND" H 3555 2927 50  0000 C CNN
 F 2 "" H 3550 3100 50  0000 C CNN
@@
 $EndComp
 $Comp
-L power-supply:GND #PWR?
+L power-supply:GND #PWR0142
 U 1 1 5E47D84D
 P 3400 3100
-F 0 "#PWR?" H 3400 2850 50  0001 C CNN
+F 0 "#PWR0142" H 3400 2850 50  0001 C CNN
 F 1 "GND" H 3405 2927 50  0000 C CNN
 F 2 "" H 3400 3100 50  0000 C CNN
@@
 	4400 1200 4500 1200
 $Comp
-L devices:INDUCTOR_SMALL L?
+L devices:INDUCTOR_SMALL L1
 U 1 1 5E40B9F0
 P 4150 1200
-F 0 "L?" H 4150 1415 50  0000 C CNN
+F 0 "L1" H 4150 1415 50  0000 C CNN
 F 1 "WE-LHMI40xx" H 4150 1324 50  0000 C CNN
 F 2 "L_power:WE-LHMI40xx" H 4150 1323 50  0001 C CNN
@@
 	3450 1200 3900 1200
 $Comp
-L devices:CP_Small C?
+L devices:CP_Small C15
 U 1 1 5E49CB58
 P 4500 1350
-F 0 "C?" H 4588 1441 50  0000 L CNN
+F 0 "C15" H 4588 1441 50  0000 L CNN
 F 1 "Tanal D" H 4500 1250 50  0000 L CNN
 F 2 "capacitors:TantalC_SizeD_EIA-7343_Wave" H 4588 1259 50  0001 L CNN
@@
 VIN_D
 $Comp
-L devices:C_1210 C?
+L devices:C_1210 C18
 U 1 1 5E5A9138
 P 6050 1800
-F 0 "C?" V 5821 1800 50  0000 C CNN
+F 0 "C18" V 5821 1800 50  0000 C CNN
 F 1 "DNI" V 5912 1800 50  0000 C CNN
 F 2 "capacitors:C_1210" H 6050 1650 50  0001 C CNN

Commit message: finished layout
Parts:
- removed C18: DNI, capacitors:C_1210, symbol devices:C_1210
- added C24: 10uF, capacitors:C_0603, symbol devices:C_0603
- added C25: 22uF, capacitors:C_0603, symbol devices:C_0603
- added U7: LT1117, SOT_TO:SOT-223, symbol voltage-regulators:LT1117
Connections:
- net +12V: no longer C12.1, C14.1, U5.2 (VIN)
- net +5V: now also C24.1, U7.3 (VIN)
- net GND: now also C15.2, C16.2, R17.2, U6.1 (GND), C24.2, C25.2, U7.1 (ADJ/GND)
- net VBAT: now also C12.1, C14.1, U5.2 (VIN)
- new net +3V3: C25.1, U7.2 (OUT), U7.4 (OUT_PAD)
Changed lines of the file:
@@
 $EndComp
 Wire Wire Line
-	2800 1200 3250 1200
+	2800 1200 2900 1200
 Wire Wire Line
 	6450 1150 6600 1150
@@
 Wire Wire Line
 	4000 2850 4000 2750
-$Comp
-L power-supply:+12V #PWR0134
-U 1 1 5E4230DE
-P 4000 2600
-F 0 "#PWR0134" H 4000 2450 50  0001 C CNN
-F 1 "+12V" H 4015 2773 50  0000 C CNN
-F 2 "" H 4000 2600 50  0000 C CNN
-F 3 "" H 4000 2600 50  0000 C CNN
-	1    4000 2600
-	1    0    0    -1
-$EndComp
 Wire Wire Line
 	4000 2850 4100 2850
@@
 	3400 2750 3550 2750
 Connection ~ 4000 2750
-Wire Wire Line
-	4000 2750 4000 2600
 Wire Wire Line
 	3550 2850 3550 2750
@@
 Text Label 3550 1200 0    50   ~ 0
 VIN_D
-$Comp
-L devices:C_1210 C18
-U 1 1 5E5A9138
-P 6050 1800
-F 0 "C18" V 5821 1800 50  0000 C CNN
-F 1 "DNI" V 5912 1800 50  0000 C CNN
-F 2 "capacitors:C_1210" H 6050 1650 50  0001 C CNN
-F 3 "" H 6050 1800 50  0000 C CNN
-	1    6050 1800
-	0    1    1    0
-$EndComp
 Wire Wire Line
 	6600 1450 6600 1800
 Wire Wire Line
-	6600 1800 6150 1800
-Wire Wire Line
 	5550 1550 5550 1800
-Wire Wire Line
-	5550 1800 5950 1800
 Connection ~ 5550 1550
 Text GLabel 2800 1200 0    50   Input ~ 0
 VBAT
+Wire Wire Line
+	5550 1800 6600 1800
+Wire Wire Line
+	2900 1200 2900 2400
+Wire Wire Line
+	2900 2400 4000 2400
+Wire Wire Line
+	4000 2400 4000 2750
+Connection ~ 2900 1200
+Wire Wire Line
+	2900 1200 3250 1200
+$Comp
+L voltage-regulators:LT1117 U7
+U 1 1 5E949600
+P 3450 6050
+F 0 "U7" H 3450 6437 60  0000 C CNN
+F 1 "LT1117" H 3450 6331 60  0000 C CNN
+F 2 "SOT_TO:SOT-223" H 3400 5750 60  0001 C CNN
+F 3 "" H 3450 6050 60  0000 C CNN
+	1    3450 6050
+	1    0    0    -1
+$EndComp
+$Comp
+L power-supply:+5V #PWR?
+U 1 1 5E94D2D6
+P 2350 5750
+F 0 "#PWR?" H 2350 5600 50  0001 C CNN
+F 1 "+5V" H 2365 5923 50  0000 C CNN
+F 2 "" H 2350 5750 50  0000 C CNN
+F 3 "" H 2350 5750 50  0000 C CNN
+	1    2350 5750
+	1    0    0    -1
+$EndComp
+$Comp
+L power-supply:+3V3 #PWR?
+U 1 1 5E94DBC1
+P 4550 5700
+F 0 "#PWR?" H 4550 5550 50  0001 C CNN
+F 1 "+3V3" H 4565 5873 50  0000 C CNN
+F 2 "" H 4550 5700 50  0000 C CNN
+F 3 "" H 4550 5700 50  0000 C CNN
+	1    4550 5700
+	1    0    0    -1
+$EndComp
+Wire Wire Line
+	4100 5950 4550 5950
+Wire Wire Line
+	4550 5950 4550 5700
+Wire Wire Line
+	4550 6100 4550 5950
+Connection ~ 4550 5950
+Wire Wire Line
+	4100 6100 4550 6100
+Wire Wire Line
+	2800 5950 2350 5950
+Wire Wire Line
+	2350 5950 2350 5750
+$Comp
+L power-supply:GND #PWR?
+U 1 1 5E95905D
+P 2700 6250
+F 0 "#PWR?" H 2700 6000 50  0001 C CNN
+F 1 "GND" H 2705 6077 50  0000 C CNN
+F 2 "" H 2700 6250 50  0000 C CNN
+F 3 "" H 2700 6250 50  0000 C CNN
+	1    2700 6250
+	1    0    0    -1
+$EndComp
+Wire Wire Line
+	2800 6100 2700 6100
+Wire Wire Line
+	2700 6100 2700 6250
+$Comp
+L devices:C_0603 C24
+U 1 1 5E961466
+P 2350 6150
+F 0 "C24" H 2442 6196 50  0000 L CNN
+F 1 "10uF" H 2442 6105 50  0000 L CNN
+F 2 "capacitors:C_0603" H 2350 6000 50  0001 C CNN
+F 3 "" H 2350 6150 50  0000 C CNN
+	1    2350 6150
+	1    0    0    -1
+$EndComp
+$Comp
+L devices:C_0603 C25
+U 1 1 5E961D25
+P 4550 6350
+F 0 "C25" H 4642 6396 50  0000 L CNN
+F 1 "22uF" H 4642 6305 50  0000 L CNN
+F 2 "capacitors:C_0603" H 4550 6200 50  0001 C CNN
+F 3 "" H 4550 6350 50  0000 C CNN
+	1    4550 6350
+	1    0    0    -1
+$EndComp
+Wire Wire Line
+	2350 6050 2350 5950
+Connection ~ 2350 5950
+Wire Wire Line
+	4550 6250 4550 6100
+Connection ~ 4550 6100
+$Comp
+L power-supply:GND #PWR?
+U 1 1 5E968467
+P 2350 6400
+F 0 "#PWR?" H 2350 6150 50  0001 C CNN
+F 1 "GND" H 2355 6227 50  0000 C CNN
+F 2 "" H 2350 6400 50  0000 C CNN
+F 3 "" H 2350 6400 50  0000 C CNN
+	1    2350 6400
+	1    0    0    -1
+$EndComp
+$Comp
+L power-supply:GND #PWR?
+U 1 1 5E9688BB
+P 4550 6600
+F 0 "#PWR?" H 4550 6350 50  0001 C CNN
+F 1 "GND" H 4555 6427 50  0000 C CNN
+F 2 "" H 4550 6600 50  0000 C CNN
+F 3 "" H 4550 6600 50  0000 C CNN
+	1    4550 6600
+	1    0    0    -1
+$EndComp
+Wire Wire Line
+	4550 6600 4550 6450
+Wire Wire Line
+	2350 6400 2350 6250
 $EndSCHEMATC

Commit message: design rules check
Parts:
- added R22: 220k, resistors:R_0603, symbol devices:R_0603
- added R23: 43.2k, resistors:R_0603, symbol devices:R_0603
Connections:
- net GND: now also R23.2
- net VBAT: now also R22.1
- net at U5.7 (EN): now also R22.2, R23.1
Changed lines of the file:
@@
-	1    0    0    -1
-$EndComp
-$Comp
-L power-supply:GND #PWR0142
-U 1 1 5E47D84D
-P 3400 3100
-F 0 "#PWR0142" H 3400 2850 50  0001 C CNN
-F 1 "GND" H 3405 2927 50  0000 C CNN
-F 2 "" H 3400 3100 50  0000 C CNN
-F 3 "" H 3400 3100 50  0000 C CNN
-	1    3400 3100
 	1    0    0    -1
 $EndComp
@@
 $EndComp
 $Comp
-L power-supply:+5V #PWR?
+L power-supply:+5V #PWR0155
 U 1 1 5E94D2D6
 P 2350 5750
-F 0 "#PWR?" H 2350 5600 50  0001 C CNN
+F 0 "#PWR0155" H 2350 5600 50  0001 C CNN
 F 1 "+5V" H 2365 5923 50  0000 C CNN
 F 2 "" H 2350 5750 50  0000 C CNN
@@
 $EndComp
 $Comp
-L power-supply:+3V3 #PWR?
+L power-supply:+3V3 #PWR0156
 U 1 1 5E94DBC1
 P 4550 5700
-F 0 "#PWR?" H 4550 5550 50  0001 C CNN
+F 0 "#PWR0156" H 4550 5550 50  0001 C CNN
 F 1 "+3V3" H 4565 5873 50  0000 C CNN
 F 2 "" H 4550 5700 50  0000 C CNN
@@
 	2350 5950 2350 5750
 $Comp
-L power-supply:GND #PWR?
+L power-supply:GND #PWR0157
 U 1 1 5E95905D
 P 2700 6250
-F 0 "#PWR?" H 2700 6000 50  0001 C CNN
+F 0 "#PWR0157" H 2700 6000 50  0001 C CNN
 F 1 "GND" H 2705 6077 50  0000 C CNN
 F 2 "" H 2700 6250 50  0000 C CNN
@@
 Connection ~ 4550 6100
 $Comp
-L power-supply:GND #PWR?
+L power-supply:GND #PWR0158
 U 1 1 5E968467
 P 2350 6400
-F 0 "#PWR?" H 2350 6150 50  0001 C CNN
+F 0 "#PWR0158" H 2350 6150 50  0001 C CNN
 F 1 "GND" H 2355 6227 50  0000 C CNN
 F 2 "" H 2350 6400 50  0000 C CNN
@@
 $EndComp
 $Comp
-L power-supply:GND #PWR?
+L power-supply:GND #PWR0159
 U 1 1 5E9688BB
 P 4550 6600
-F 0 "#PWR?" H 4550 6350 50  0001 C CNN
+F 0 "#PWR0159" H 4550 6350 50  0001 C CNN
 F 1 "GND" H 4555 6427 50  0000 C CNN
 F 2 "" H 4550 6600 50  0000 C CNN
@@
 Wire Wire Line
 	2350 6400 2350 6250
+$Comp
+L devices:R_0603 R22
+U 1 1 5E9848CE
+P 1300 2550
+F 0 "R22" H 1359 2596 50  0000 L CNN
+F 1 "220k" H 1359 2505 50  0000 L CNN
+F 2 "resistors:R_0603" H 1300 2400 50  0001 C CNN
+F 3 "" H 1300 2550 50  0000 C CNN
+	1    1300 2550
+	1    0    0    -1
+$EndComp
+$Comp
+L devices:R_0603 R23
+U 1 1 5E984E13
+P 1300 3000
+F 0 "R23" H 1359 3046 50  0000 L CNN
+F 1 "43.2k" H 1359 2955 50  0000 L CNN
+F 2 "resistors:R_0603" H 1300 2850 50  0001 C CNN
+F 3 "" H 1300 3000 50  0000 C CNN
+	1    1300 3000
+	1    0    0    -1
+$EndComp
+Wire Wire Line
+	2150 2800 1300 2800
+Wire Wire Line
+	1300 2800 1300 2900
+Wire Wire Line
+	1300 2800 1300 2650
+Connection ~ 1300 2800
+Text GLabel 1300 2300 1    50   Input ~ 0
+VBAT
+$Comp
+L power-supply:GND #PWR0160
+U 1 1 5E99D5C7
+P 1300 3300
+F 0 "#PWR0160" H 1300 3050 50  0001 C CNN
+F 1 "GND" H 1305 3127 50  0000 C CNN
+F 2 "" H 1300 3300 50  0000 C CNN
+F 3 "" H 1300 3300 50  0000 C CNN
+	1    1300 3300
+	1    0    0    -1
+$EndComp
+Wire Wire Line
+	1300 2450 1300 2300
+Wire Wire Line
+	1300 3300 1300 3100
+Wire Wire Line
+	3400 3100 3550 3100
+Connection ~ 3550 3100
+Wire Wire Line
+	4100 3100 3950 3100
+Wire Wire Line
+	3950 3100 3950 3250
+Wire Wire Line
+	3950 3250 2150 3250
+Wire Wire Line
+	2150 2800 2150 3250
 $EndSCHEMATC
