File: hardware/controlpcb/kicad/connectors.sch (KiCad schematic (older format))
At the start: 20 parts, among them P1 USB_B, U2 BSS138, U3 BSS138

Commit message: fixed layout and created case
Connections:
- net GND: now also BAT1.2 (P2)
Changed lines of the file:
@@
 L power-supply:GND #PWR0154
 U 1 1 5E98D818
-P 8750 4900
-F 0 "#PWR0154" H 8750 4650 50  0001 C CNN
-F 1 "GND" H 8755 4727 50  0000 C CNN
-F 2 "" H 8750 4900 50  0000 C CNN
-F 3 "" H 8750 4900 50  0000 C CNN
-	1    8750 4900
+P 8800 4900
+F 0 "#PWR0154" H 8800 4650 50  0001 C CNN
+F 1 "GND" H 8805 4727 50  0000 C CNN
+F 2 "" H 8800 4900 50  0000 C CNN
+F 3 "" H 8800 4900 50  0000 C CNN
+	1    8800 4900
 	1    0    0    -1
 $EndComp
@@
 	8750 4600 9350 4600
 Wire Wire Line
-	9300 4700 8750 4700
+	9350 4700 8800 4700
 Wire Wire Line
-	8750 4700 8750 4900
+	8800 4700 8800 4900
 $EndSCHEMATC
